Commit message: Add PBR materials with HDR environment mapping
Refactor URDF viewer to use physically-based rendering with environment maps for realistic reflections. Convert legacy materials (Phong/Lambert/Basic) to MeshStandardMaterial with quarry HDR environment.

- Add HDR environment map loading with PMREM preprocessing
- Auto-convert legacy materials to PBR with proper envMap handling
- Fix dual Three.js bundle issues using type string checks
- Add tone mapping for proper HDR display
- Refactor viewer code for better maintainability
- Add Collada (.dae) mesh support

🤖 Generated with [Claude Code](https://claude.com/claude-code)

Co-Authored-By: Claude <noreply@anthropic.com>

File: urdf/yam/urdf/yam.urdf (robot description, URDF)
Before this commit: robot yam_v0, 7 links, 6 joints
Links:
- link base_link: geometry collision mesh filename=../meshes/base_link_collision.stl; visual mesh filename=../meshes/base_link_visual.dae
- link link_1: geometry collision mesh filename=../meshes/link_1_collision.stl; visual mesh filename=../meshes/link_1_visual.dae
- link link_2: geometry collision mesh filename=../meshes/link_2_collision.stl; visual mesh filename=../meshes/link_2_visual.dae
- link link_3: geometry collision mesh filename=../meshes/link_3_collision.stl; visual mesh filename=../meshes/link_3_visual.dae
- link link_4: geometry collision mesh filename=../meshes/link_4_collision.stl; visual mesh filename=../meshes/link_4_visual.dae
- link link_5: geometry collision mesh filename=../meshes/link_5_collision.stl; visual mesh filename=../meshes/link_5_visual.dae
- link link_6: geometry collision mesh filename=../meshes/link_6_collision.stl; visual mesh filename=../meshes/link_6_visual.dae
